File: Debug_Port.sch (EAGLE design)
At the start: 16 parts, among them J1 QSH-030-01-X-D-A

Commit message: Iteration on companion board.
Parts:
- added JP10: ADAFRUIT BMP280 Breakout, pinhead:PINHD-1X7
- added Q1: CSM-7X-DU, crystal:CSM-7X-DU
- added R2: 0k, resistor:R-US_R0805
- added R3: 10k, resistor:R-US_R0805
- JP8: device pinhead:PINHD-2X5 -> pinhead:PINHD-2X7
- U$1: value (none) -> MSP430FR2311IPW20; device parts:MSP430FR2311IPW16 -> companion_board:MSP430FR2311IPW20
Connections:
- net BSL_TEST renamed SBW_TEST
- removed net BSL_RST: JP8.4, R1.1, U$1.RST/NMI/SBWTDIO
- removed net BSL_RX: JP8.3
- removed net BSL_TCK: JP8.2
- removed net BSL_TX: JP8.1
- removed net BSL_VCC: JP8.6, JP9.1
- removed net BSL_VCC_SENSE: JP8.8
- removed net N$50: U$1.P1.7/UCA0TXD/UCA0SIMO/TB0.2/TDO/TRI0+/A7/VREF+
- new net BSL_RXD: JP8.12, U$1.P1.6/UCA0RXD/UCA0SOMI/TB0.1/TDI/TCLK/TRI0-/A6
- new net BSL_TXD: JP8.14, U$1.P1.7/UCA-TXD/UCA0SIMO/TB0.2/TDO/TRI0+/A7/VREF+
- new net DISABLE_DEADMAN: R2.1, R3.1, U$1.P1.1/UCB0CLK/ACLK/C1/A1
- new net LIGHT_PWM1: U$1.P2.0/TB1.1/COUT
- new net LIGHT_PWM2: U$1.P2.1/TB1.2
- new net SBW_RST: JP8.1, R1.1, U$1.RST/NMI/SBWTDIO
- new net VCC_TARGET: JP8.4, JP9.1
- new net VCC_TOOL: JP8.2, JP9.3
- new net XBEE_DIO0: R2.2, XB1.AD0/DIO0
- net +3V3: now also JP10.2, JP10.7, JP9.2, R1.2, R3.2, U$1.DVCC; no longer JP9.3
- net GND: now also JP10.3, JP10.5, JP8.9; no longer JP8.5
- net I2C_GP0_CLK_3V3: now also U$1.P1.3/UCB0SOMI/UCB0SCL/OA0O/A3
- net I2C_GP0_DAT_3V3: now also JP10.6, U$1.P1.2/UCB0SIMO/UCB0SDA/TB0TRG/OA0-/A2/VEREF-
- net N$41: now also Q1.2, U$1.P2.7/TB0CLK/XIN; no longer U$1.P1.6/UCA0RXD/UCA0SOMI/TB0.1/TDI/TCLK/A6
- net N$47: now also Q1.1, U$1.P2.6/MCLK/XOUT; no longer JP9.2, R1.2, U$1.DVCC
Other:
- note added: "3V3"
- note added: "ADR"
- note added: "CS"
- note added: "GND"
- note added: "Grounding ADR sets I2C addr to 0x76"
- note added: "SCL"
- note added: "SDA"
- moved on the sheet: JP9
