File: Companion_Board.sch (EAGLE design)
At the start: 34 parts, among them J1 QSH-030-01-X-D-A, Q1 CSM-7X-DU

Commit message: Changed name to Companion_Board
Parts:
- JP12: value (none) -> PWM Light Control
Other:
- moved on the sheet: JP6, JP7
Changed lines of the file:
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@@
 <part name="TP2" library="testpad" deviceset="TP" device="PAD1-13"/>
 <part name="TP3" library="testpad" deviceset="TP" device="PAD1-13"/>
-<part name="JP12" library="pinhead" deviceset="PINHD-1X3" device="/90"/>
+<part name="JP12" library="pinhead" deviceset="PINHD-1X3" device="/90" value="PWM Light Control"/>
 <part name="SUPPLY15" library="supply2" deviceset="GND" device=""/>
 <part name="JP13" library="pinhead" deviceset="PINHD-1X10" device=""/>
@@
 <instance part="P+3" gate="VCC" x="269.24" y="5.08"/>
 <instance part="JP4" gate="A" x="124.46" y="-40.64"/>
-<instance part="JP6" gate="A" x="27.94" y="50.8" rot="MR0"/>
-<instance part="JP7" gate="A" x="180.34" y="53.34"/>
+<instance part="JP6" gate="A" x="40.64" y="50.8" rot="MR0"/>
+<instance part="JP7" gate="A" x="172.72" y="53.34"/>
 <instance part="XB1" gate="G$1" x="383.54" y="60.96"/>
 <instance part="+3V4" gate="G$1" x="358.14" y="114.3"/>
@@
 <wire x1="50.8" y1="93.98" x2="50.8" y2="55.88" width="0.1524" layer="91"/>
 <pinref part="JP6" gate="A" pin="3"/>
-<wire x1="50.8" y1="55.88" x2="30.48" y2="55.88" width="0.1524" layer="91"/>
+<wire x1="50.8" y1="55.88" x2="43.18" y2="55.88" width="0.1524" layer="91"/>
 </segment>
 </net>
@@
 <junction x="78.74" y="30.48"/>
 <pinref part="JP6" gate="A" pin="2"/>
-<wire x1="30.48" y1="58.42" x2="53.34" y2="58.42" width="0.1524" layer="91"/>
+<wire x1="43.18" y1="58.42" x2="53.34" y2="58.42" width="0.1524" layer="91"/>
 <wire x1="53.34" y1="58.42" x2="53.34" y2="91.44" width="0.1524" layer="91"/>
 <wire x1="53.34" y1="91.44" x2="78.74" y2="91.44" width="0.1524" layer="91"/>
 <junction x="78.74" y="91.44"/>
 <pinref part="JP6" gate="A" pin="10"/>
-<wire x1="30.48" y1="38.1" x2="63.5" y2="38.1" width="0.1524" layer="91"/>
+<wire x1="43.18" y1="38.1" x2="63.5" y2="38.1" width="0.1524" layer="91"/>
 <wire x1="63.5" y1="38.1" x2="63.5" y2="22.86" width="0.1524" layer="91"/>
 <wire x1="63.5" y1="22.86" x2="78.74" y2="22.86" width="0.1524" layer="91"/>
@@
 <junction x="63.5" y="38.1"/>
 <pinref part="JP6" gate="A" pin="9"/>
-<wire x1="63.5" y1="40.64" x2="30.48" y2="40.64" width="0.1524" layer="91"/>
+<wire x1="63.5" y1="40.64" x2="43.18" y2="40.64" width="0.1524" layer="91"/>
 </segment>
 <segment>
@@
 <wire x1="160.02" y1="91.44" x2="160.02" y2="68.58" width="0.1524" layer="91"/>
 <pinref part="JP7" gate="A" pin="2"/>
-<wire x1="160.02" y1="68.58" x2="177.8" y2="68.58" width="0.1524" layer="91"/>
+<wire x1="160.02" y1="68.58" x2="170.18" y2="68.58" width="0.1524" layer="91"/>
 <wire x1="114.3" y1="22.86" x2="160.02" y2="22.86" width="0.1524" layer="91"/>
 <wire x1="160.02" y1="22.86" x2="160.02" y2="35.56" width="0.1524" layer="91"/>
 <pinref part="JP7" gate="A" pin="15"/>
-<wire x1="160.02" y1="35.56" x2="177.8" y2="35.56" width="0.1524" layer="91"/>
+<wire x1="160.02" y1="35.56" x2="170.18" y2="35.56" width="0.1524" layer="91"/>
 </segment>
 <segment>
@@
 <wire x1="144.78" y1="45.72" x2="144.78" y2="50.8" width="0.1524" layer="91"/>
 <pinref part="JP7" gate="A" pin="9"/>
-<wire x1="144.78" y1="50.8" x2="177.8" y2="50.8" width="0.1524" layer="91"/>
+<wire x1="144.78" y1="50.8" x2="170.18" y2="50.8" width="0.1524" layer="91"/>
 </segment>
 <segment>
 <pinref part="JP7" gate="A" pin="11"/>
-<wire x1="177.8" y1="45.72" x2="149.86" y2="45.72" width="0.1524" layer="91"/>
+<wire x1="170.18" y1="45.72" x2="149.86" y2="45.72" width="0.1524" layer="91"/>
 <wire x1="149.86" y1="45.72" x2="149.86" y2="40.64" width="0.1524" layer="91"/>
 <pinref part="J1" gate="G$1" pin="44"/>
@@
 <wire x1="152.4" y1="38.1" x2="152.4" y2="43.18" width="0.1524" layer="91"/>
 <pinref part="JP7" gate="A" pin="12"/>
-<wire x1="152.4" y1="43.18" x2="177.8" y2="43.18" width="0.1524" layer="91"/>
+<wire x1="152.4" y1="43.18" x2="170.18" y2="43.18" width="0.1524" layer="91"/>
 </segment>
 <segment>
@@
 <wire x1="147.32" y1="76.2" x2="147.32" y2="55.88" width="0.1524" layer="91"/>
 <pinref part="JP7" gate="A" pin="7"/>
-<wire x1="147.32" y1="55.88" x2="177.8" y2="55.88" width="0.1524" layer="91"/>
+<wire x1="147.32" y1="55.88" x2="170.18" y2="55.88" width="0.1524" layer="91"/>
 </segment>
 </net>
@@
 <label x="119.38" y="73.66" size="1.778" layer="95"/>
 <pinref part="JP7" gate="A" pin="8"/>
-<wire x1="177.8" y1="53.34" x2="144.78" y2="53.34" width="0.1524" layer="91"/>
+<wire x1="170.18" y1="53.34" x2="144.78" y2="53.34" width="0.1524" layer="91"/>
 <wire x1="144.78" y1="53.34" x2="144.78" y2="73.66" width="0.1524" layer="91"/>
 <wire x1="144.78" y1="73.66" x2="109.22" y2="73.66" width="0.1524" layer="91"/>
@@
 <wire x1="162.56" y1="93.98" x2="162.56" y2="71.12" width="0.1524" layer="91"/>
 <pinref part="JP7" gate="A" pin="1"/>
-<wire x1="162.56" y1="71.12" x2="177.8" y2="71.12" width="0.1524" layer="91"/>
+<wire x1="162.56" y1="71.12" x2="170.18" y2="71.12" width="0.1524" layer="91"/>
 </segment>
 <segment>
@@
 <label x="58.42" y="68.58" size="1.778" layer="95"/>
 <pinref part="JP6" gate="A" pin="1"/>
-<wire x1="30.48" y1="60.96" x2="55.88" y2="60.96" width="0.1524" layer="91"/>
+<wire x1="43.18" y1="60.96" x2="55.88" y2="60.96" width="0.1524" layer="91"/>
 </segment>
 </net>
@@
 <wire x1="154.94" y1="27.94" x2="154.94" y2="40.64" width="0.1524" layer="91"/>
 <pinref part="JP7" gate="A" pin="13"/>
-<wire x1="154.94" y1="40.64" x2="177.8" y2="40.64" width="0.1524" layer="91"/>
+<wire x1="154.94" y1="40.64" x2="170.18" y2="40.64" width="0.1524" layer="91"/>
 </segment>
 </net>
@@
 <wire x1="157.48" y1="25.4" x2="157.48" y2="38.1" width="0.1524" layer="91"/>
 <pinref part="JP7" gate="A" pin="14"/>
-<wire x1="157.48" y1="38.1" x2="177.8" y2="38.1" width="0.1524" layer="91"/>
+<wire x1="157.48" y1="38.1" x2="170.18" y2="38.1" width="0.1524" layer="91"/>
 </segment>
 </net>
@@
 <wire x1="58.42" y1="66.04" x2="58.42" y2="53.34" width="0.1524" layer="91"/>
 <pinref part="JP6" gate="A" pin="4"/>
-<wire x1="58.42" y1="53.34" x2="30.48" y2="53.34" width="0.1524" layer="91"/>
+<wire x1="58.42" y1="53.34" x2="43.18" y2="53.34" width="0.1524" layer="91"/>
 <label x="60.96" y="66.04" size="1.778" layer="95"/>
 </segment>
@@
 <segment>
 <pinref part="JP6" gate="A" pin="5"/>
-<wire x1="30.48" y1="50.8" x2="60.96" y2="50.8" width="0.1524" layer="91"/>
+<wire x1="43.18" y1="50.8" x2="60.96" y2="50.8" width="0.1524" layer="91"/>
 <wire x1="60.96" y1="50.8" x2="60.96" y2="63.5" width="0.1524" layer="91"/>
 <pinref part="J1" gate="G$1" pin="25"/>
@@
 <wire x1="63.5" y1="60.96" x2="63.5" y2="48.26" width="0.1524" layer="91"/>
 <pinref part="JP6" gate="A" pin="6"/>
-<wire x1="63.5" y1="48.26" x2="30.48" y2="48.26" width="0.1524" layer="91"/>
+<wire x1="63.5" y1="48.26" x2="43.18" y2="48.26" width="0.1524" layer="91"/>
 <label x="66.04" y="60.96" size="1.778" layer="95"/>
 </segment>
@@
 <segment>
 <pinref part="JP6" gate="A" pin="7"/>
-<wire x1="30.48" y1="45.72" x2="66.04" y2="45.72" width="0.1524" layer="91"/>
+<wire x1="43.18" y1="45.72" x2="66.04" y2="45.72" width="0.1524" layer="91"/>
 <wire x1="66.04" y1="45.72" x2="66.04" y2="58.42" width="0.1524" layer="91"/>
 <pinref part="J1" gate="G$1" pin="29"/>
@@
 <wire x1="66.04" y1="25.4" x2="66.04" y2="43.18" width="0.1524" layer="91"/>
 <pinref part="JP6" gate="A" pin="8"/>
-<wire x1="66.04" y1="43.18" x2="30.48" y2="43.18" width="0.1524" layer="91"/>
+<wire x1="66.04" y1="43.18" x2="43.18" y2="43.18" width="0.1524" layer="91"/>
 <label x="66.04" y="25.4" size="1.778" layer="95"/>
 </segment>
@@
 <wire x1="157.48" y1="88.9" x2="157.48" y2="66.04" width="0.1524" layer="91"/>
 <pinref part="JP7" gate="A" pin="3"/>
-<wire x1="157.48" y1="66.04" x2="177.8" y2="66.04" width="0.1524" layer="91"/>
+<wire x1="157.48" y1="66.04" x2="170.18" y2="66.04" width="0.1524" layer="91"/>
 <label x="119.38" y="88.9" size="1.778" layer="95"/>
 </segment>
@@
 <segment>
 <pinref part="JP7" gate="A" pin="4"/>
-<wire x1="177.8" y1="63.5" x2="154.94" y2="63.5" width="0.1524" layer="91"/>
+<wire x1="170.18" y1="63.5" x2="154.94" y2="63.5" width="0.1524" layer="91"/>
 <wire x1="154.94" y1="63.5" x2="154.94" y2="86.36" width="0.1524" layer="91"/>
 <pinref part="J1" gate="G$1" pin="8"/>
@@
 <wire x1="152.4" y1="83.82" x2="152.4" y2="60.96" width="0.1524" layer="91"/>
 <pinref part="JP7" gate="A" pin="5"/>
-<wire x1="152.4" y1="60.96" x2="177.8" y2="60.96" width="0.1524" layer="91"/>
+<wire x1="152.4" y1="60.96" x2="170.18" y2="60.96" width="0.1524" layer="91"/>
 <label x="119.38" y="83.82" size="1.778" layer="95"/>
 </segment>
@@
 <segment>
 <pinref part="JP7" gate="A" pin="6"/>
-<wire x1="177.8" y1="58.42" x2="149.86" y2="58.42" width="0.1524" layer="91"/>
+<wire x1="170.18" y1="58.42" x2="149.86" y2="58.42" width="0.1524" layer="91"/>
 <wire x1="149.86" y1="58.42" x2="149.86" y2="81.28" width="0.1524" layer="91"/>
 <pinref part="J1" gate="G$1" pin="12"/>
@@
 <wire x1="147.32" y1="43.18" x2="147.32" y2="48.26" width="0.1524" layer="91"/>
 <pinref part="JP7" gate="A" pin="10"/>
-<wire x1="147.32" y1="48.26" x2="177.8" y2="48.26" width="0.1524" layer="91"/>
+<wire x1="147.32" y1="48.26" x2="170.18" y2="48.26" width="0.1524" layer="91"/>
 <label x="119.38" y="43.18" size="1.778" layer="95"/>
 </segment>

Commit message: Working on Companion board and README.
Parts:
- added D1, D2: RED, SparkFun-LED:LED-RED1206
- added R6, R7, R8, R9: 10k, resistor:R-US_R0805
- added U$3, U$4: 2N7002DW, companion_board:2N7002DW
Connections:
- removed net N$50: JP11.7, U$1.P2.5/UCB0SOMI/USB0SCL
- removed net N$53: JP11.9, U$1.P2.4/UCB0SIMO/UCB0SDA
- new net MSP_LED1: JP11.7, R8.1, U$1.P2.5/UCB0SOMI/USB0SCL, U$4G$1.G
- new net MSP_LED2: JP11.9, R6.1, U$1.P2.4/UCB0SIMO/UCB0SDA, U$3G$1.G
- new net N$69: D1.C, U$3G$1.D
- new net N$70: D1.A, R7.1
- new net N$72: D2.C, U$4G$1.D
- new net N$73: D2.A, R9.1
- net +3V3: now also R7.2, R9.2
- net GND: now also R6.2, R8.2, U$3G$1.S, U$4G$1.S
Changed lines of the file:
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@@
 <part name="FRAME1" library="frames" deviceset="FRAME_B_L" device=""/>
 <part name="SUPPLY19" library="supply2" deviceset="GND" device=""/>
+<part name="U$3" library="companion_board" deviceset="2N7002DW" device=""/>
+<part name="SUPPLY20" library="supply2" deviceset="GND" device=""/>
+<part name="R6" library="resistor" deviceset="R-US_" device="R0805" value="10k"/>
+<part name="D1" library="SparkFun-LED" deviceset="LED-RED" device="1206" value="RED"/>
+<part name="R7" library="resistor" deviceset="R-US_" device="R0805" value="10k"/>
+<part name="U$4" library="companion_board" deviceset="2N7002DW" device=""/>
+<part name="SUPPLY21" library="supply2" deviceset="GND" device=""/>
+<part name="R8" library="resistor" deviceset="R-US_" device="R0805" value="10k"/>
+<part name="D2" library="SparkFun-LED" deviceset="LED-RED" device="1206" value="RED"/>
+<part name="R9" library="resistor" deviceset="R-US_" device="R0805" value="10k"/>
+<part name="+3V8" library="supply1" deviceset="+3V3" device=""/>
 </parts>
 <sheets>
@@
 <instance part="FRAME1" gate="G$2" x="342.9" y="-60.96"/>
 <instance part="SUPPLY19" gate="GND" x="309.88" y="91.44"/>
+<instance part="U$3" gate="G$1" x="119.38" y="116.84" rot="MR0"/>
+<instance part="SUPPLY20" gate="GND" x="114.3" y="106.68" rot="MR0"/>
+<instance part="R6" gate="G$1" x="121.92" y="109.22" rot="MR0"/>
+<instance part="D1" gate="G$1" x="114.3" y="124.46"/>
+<instance part="R7" gate="G$1" x="114.3" y="132.08" rot="R90"/>
+<instance part="U$4" gate="G$1" x="71.12" y="116.84" rot="MR0"/>
+<instance part="SUPPLY21" gate="GND" x="66.04" y="106.68" rot="MR0"/>
+<instance part="R8" gate="G$1" x="73.66" y="109.22" rot="MR0"/>
+<instance part="D2" gate="G$1" x="66.04" y="124.46"/>
+<instance part="R9" gate="G$1" x="66.04" y="132.08" rot="R90"/>
+<instance part="+3V8" gate="G$1" x="66.04" y="139.7"/>
 </instances>
 <busses>
@@
 <wire x1="322.58" y1="15.24" x2="322.58" y2="20.32" width="0.1524" layer="91"/>
 </segment>
+<segment>
+<pinref part="U$3" gate="G$1" pin="S"/>
+<pinref part="SUPPLY20" gate="GND" pin="GND"/>
+<wire x1="114.3" y1="114.3" x2="114.3" y2="109.22" width="0.1524" layer="91"/>
+<pinref part="R6" gate="G$1" pin="2"/>
+<wire x1="116.84" y1="109.22" x2="114.3" y2="109.22" width="0.1524" layer="91"/>
+<junction x="114.3" y="109.22"/>
+</segment>
+<segment>
+<pinref part="U$4" gate="G$1" pin="S"/>
+<pinref part="SUPPLY21" gate="GND" pin="GND"/>
+<wire x1="66.04" y1="114.3" x2="66.04" y2="109.22" width="0.1524" layer="91"/>
+<pinref part="R8" gate="G$1" pin="2"/>
+<wire x1="68.58" y1="109.22" x2="66.04" y2="109.22" width="0.1524" layer="91"/>
+<junction x="66.04" y="109.22"/>
+</segment>
 </net>
 <net name="RESET_IN_R_L" class="0">
@@
 <wire x1="213.36" y1="132.08" x2="220.98" y2="132.08" width="0.1524" layer="91"/>
 </segment>
+<segment>
+<pinref part="R9" gate="G$1" pin="2"/>
+<pinref part="+3V8" gate="G$1" pin="+3V3"/>
+<pinref part="R7" gate="G$1" pin="2"/>
+<wire x1="66.04" y1="137.16" x2="114.3" y2="137.16" width="0.1524" layer="91"/>
+<junction x="66.04" y="137.16"/>
+</segment>
 </net>
 <net name="+5V" class="0">
@@
 <pinref part="JP8" gate="A" pin="7"/>
 <wire x1="66.04" y1="160.02" x2="45.72" y2="160.02" width="0.1524" layer="91"/>
-<wire x1="45.72" y1="160.02" x2="45.72" y2="137.16" width="0.1524" layer="91"/>
-<wire x1="45.72" y1="137.16" x2="114.3" y2="137.16" width="0.1524" layer="91"/>
-<wire x1="114.3" y1="137.16" x2="114.3" y2="162.56" width="0.1524" layer="91"/>
+<wire x1="45.72" y1="160.02" x2="45.72" y2="144.78" width="0.1524" layer="91"/>
+<wire x1="45.72" y1="144.78" x2="114.3" y2="144.78" width="0.1524" layer="91"/>
+<wire x1="114.3" y1="144.78" x2="114.3" y2="162.56" width="0.1524" layer="91"/>
 <pinref part="U$1" gate="G$1" pin="TEST/SBWTCK"/>
 </segment>
@@
 </segment>
 </net>
-<net name="N$50" class="0">
+<net name="MSP_LED1" class="0">
 <segment>
 <pinref part="U$1" gate="G$1" pin="P2.5/UCB0SOMI/USB0SCL"/>
@@
 <pinref part="JP11" gate="A" pin="7"/>
 <wire x1="170.18" y1="124.46" x2="220.98" y2="124.46" width="0.1524" layer="91"/>
-</segment>
-</net>
-<net name="N$53" class="0">
-<segment>
-<pinref part="U$1" gate="G$1" pin="P2.4/UCB0SIMO/UCB0SDA"/>
-<wire x1="175.26" y1="144.78" x2="172.72" y2="144.78" width="0.1524" layer="91"/>
-<wire x1="172.72" y1="144.78" x2="172.72" y2="121.92" width="0.1524" layer="91"/>
-<pinref part="JP11" gate="A" pin="9"/>
-<wire x1="172.72" y1="121.92" x2="220.98" y2="121.92" width="0.1524" layer="91"/>
+<label x="177.8" y="124.46" size="1.778" layer="95"/>
+</segment>
+<segment>
+<pinref part="U$4" gate="G$1" pin="G"/>
+<wire x1="76.2" y1="114.3" x2="81.28" y2="114.3" width="0.1524" layer="91"/>
+<wire x1="81.28" y1="114.3" x2="81.28" y2="109.22" width="0.1524" layer="91"/>
+<pinref part="R8" gate="G$1" pin="1"/>
+<wire x1="78.74" y1="109.22" x2="81.28" y2="109.22" width="0.1524" layer="91"/>
+<junction x="81.28" y="114.3"/>
+<wire x1="81.28" y1="114.3" x2="101.6" y2="114.3" width="0.1524" layer="91"/>
+<label x="86.36" y="114.3" size="1.778" layer="95"/>
 </segment>
 </net>
@@
 </segment>
 </net>
+<net name="MSP_LED2" class="0">
+<segment>
+<pinref part="U$3" gate="G$1" pin="G"/>
+<wire x1="124.46" y1="114.3" x2="129.54" y2="114.3" width="0.1524" layer="91"/>
+<wire x1="129.54" y1="114.3" x2="129.54" y2="109.22" width="0.1524" layer="91"/>
+<pinref part="R6" gate="G$1" pin="1"/>
+<wire x1="127" y1="109.22" x2="129.54" y2="109.22" width="0.1524" layer="91"/>
+<junction x="129.54" y="114.3"/>
+<pinref part="U$1" gate="G$1" pin="P2.4/UCB0SIMO/UCB0SDA"/>
+<wire x1="175.26" y1="144.78" x2="172.72" y2="144.78" width="0.1524" layer="91"/>
+<wire x1="172.72" y1="144.78" x2="172.72" y2="121.92" width="0.1524" layer="91"/>
+<pinref part="JP11" gate="A" pin="9"/>
+<wire x1="172.72" y1="121.92" x2="220.98" y2="121.92" width="0.1524" layer="91"/>
+<wire x1="129.54" y1="114.3" x2="172.72" y2="114.3" width="0.1524" layer="91"/>
+<wire x1="172.72" y1="114.3" x2="172.72" y2="121.92" width="0.1524" layer="91"/>
+<junction x="172.72" y="121.92"/>
+<label x="134.62" y="114.3" size="1.778" layer="95"/>
+<label x="177.8" y="121.92" size="1.778" layer="95"/>
+</segment>
+</net>
+<net name="N$69" class="0">
+<segment>
+<pinref part="U$3" gate="G$1" pin="D"/>
+<pinref part="D1" gate="G$1" pin="C"/>
+</segment>
+</net>
+<net name="N$70" class="0">
+<segment>
+<pinref part="D1" gate="G$1" pin="A"/>
+<pinref part="R7" gate="G$1" pin="1"/>
+</segment>
+</net>
+<net name="N$72" class="0">
+<segment>
+<pinref part="U$4" gate="G$1" pin="D"/>
+<pinref part="D2" gate="G$1" pin="C"/>
+</segment>
+</net>
+<net name="N$73" class="0">
+<segment>
+<pinref part="D2" gate="G$1" pin="A"/>
+<pinref part="R9" gate="G$1" pin="1"/>
+</segment>
+</net>

Commit message: Consolidating footprints for companion board.
Parts:
- removed JP11: (no value), pinhead:PINHD-2X5
- added R10: 10k, resistor:R-US_R0805
- added R11: 0k, resistor:R-US_R0805
- R7, R9: value 10k -> ??k
- renumbered J1 to J10, SV1 to J26, SV2 to J17, SV3 to J21
Connections:
- net I2C_GP2_CLK_3V3 renamed I2C_GP1_CLK_3V3_J10
- removed net N$34: J21.27, JP3.14
- removed net N$48: JP11.5, U$1.P1.0/UCB0STE/SMCLK/C0/A0/VEREF+
- removed net N$68: JP14.9, XB1.AD1/DIO1
- new net I2C_GP1_DAT_3V3_J10: J10.56, JP7.14
- new net XBEE_DIO1: JP14.9, R11.2, XB1.AD1/DIO1
- net +3V3: now also R10.2; no longer JP11.1
- net DISABLE_DEADMAN: now also R10.1; no longer JP11.3, R3.1
- net GND: now also J26.10, JP2.5; no longer JP11.10
- net I2C_GP1_DAT_3V3: now also J21.27, JP3.14; no longer J10.56, JP7.14
- net MSP_LED1: no longer JP11.7
- net MSP_LED2: no longer JP11.9
- net N$25: now also R11.1, R3.1, U$1.P1.0/UCB0STE/SMCLK/C0/A0/VEREF+; no longer J26.10, JP2.5
- net N$54: no longer JP11.2
- net N$55: no longer JP11.4
- net N$56: no longer JP11.6
- net N$57: no longer JP11.8
Other:
- note added: "J10: Debug Connector"
- note added: "J17: UART Connector"
- note added: "J21: Expansion Header"
- note added: "J26: GPIO Expansion Header"
- note added: "SEG IRD FY2016 Stereo Camera: Jetson TX1 Companion Board"
- note removed: "Debug Connector"
- note removed: "Expansion Header"
- note removed: "GPIO Expansion Header"
- note removed: "UART Connector"
- moved on the sheet: C1, C3, R1, R2, R3
